File: schema/Robothond/Robothond.sch (KiCad schematic (older format))
At the start: 8 parts

Commit message: added SVG of schema
Parts:
- U1: renamed from U?; symbol L298N:L298N -> Robothond-rescue:L298N-L298N
- U2, U3, U4: renamed from U?; symbol HC-SR04:HC-SR04 -> Robothond-rescue:HC-SR04-HC-SR04
- gave numbers to parts that had none: 4
Other:
- moved on the sheet: A1, BT1, M1, M2, U1, U2, U3, U4
