File: schema/Robothond/Robothond.kicad_sch (KiCad schematic)
At the start: 8 parts

Commit message: Changed name into initials
Parts:
- A1: value (none) -> Arduino_Leonardo; footprint (none) -> Module:Arduino_UNO_R3
- BT1: value (none) -> Battery
- M1, M2: value (none) -> Motor_DC
- U1: value (none) -> L298N; footprint (none) -> TO127P2020X500X2100-15
- U2, U3, U4: value (none) -> HC-SR04; footprint (none) -> XCVR_HC-SR04
Changed lines of the file:
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@@
     (title "Aansluitschema Robothond")
     (date "2022-05-24")
-    (rev "IJdo IJssennagger")
+    (rev "IJ. IJ.")
     (comment 1 "Christian Wanschers, IJdo IJssennagger, Kris Boogert")
     (comment 2 "Aansluitschema gerealiseerd door:")
@@
     (in_bom yes) (on_board yes)
     (property "Reference" "A1" (id 0) (at 168.91 61.4426 0))
-    (property "Value" "" (id 1) (at 168.91 63.754 0))
-    (property "Footprint" "" (id 2) (at 168.91 91.44 0)
+    (property "Value" "Arduino_Leonardo" (id 1) (at 168.91 63.754 0))
+    (property "Footprint" "Module:Arduino_UNO_R3" (id 2) (at 168.91 91.44 0)
       (effects (font (size 1.27 1.27) italic) hide)
     )
@@
     (in_bom yes) (on_board yes)
     (property "Reference" "U1" (id 0) (at 129.54 74.549 0))
-    (property "Value" "" (id 1) (at 129.54 76.8604 0))
-    (property "Footprint" "" (id 2) (at 129.54 96.52 0)
+    (property "Value" "L298N" (id 1) (at 129.54 76.8604 0))
+    (property "Footprint" "TO127P2020X500X2100-15" (id 2) (at 129.54 96.52 0)
       (effects (font (size 1.27 1.27)) (justify left bottom) hide)
     )
@@
     (in_bom yes) (on_board yes)
     (property "Reference" "BT1" (id 0) (at 96.52 73.787 90))
-    (property "Value" "" (id 1) (at 96.52 76.0984 90))
+    (property "Value" "Battery" (id 1) (at 96.52 76.0984 90))
     (property "Footprint" "" (id 2) (at 98.044 80.01 90)
       (effects (font (size 1.27 1.27)) hide)
@@
     (in_bom yes) (on_board yes)
     (property "Reference" "M2" (id 0) (at 96.52 101.727 90))
-    (property "Value" "" (id 1) (at 96.52 104.0384 90))
+    (property "Value" "Motor_DC" (id 1) (at 96.52 104.0384 90))
     (property "Footprint" "" (id 2) (at 95.504 109.22 0)
       (effects (font (size 1.27 1.27)) hide)
@@
     (in_bom yes) (on_board yes)
     (property "Reference" "M1" (id 0) (at 96.52 86.487 90))
-    (property "Value" "" (id 1) (at 96.52 88.7984 90))
+    (property "Value" "Motor_DC" (id 1) (at 96.52 88.7984 90))
     (property "Footprint" "" (id 2) (at 95.504 93.98 0)
       (effects (font (size 1.27 1.27)) hide)
@@
       (effects (font (size 1.27 1.27)) (justify left))
     )
-    (property "Value" "" (id 1) (at 216.662 82.423 0)
-      (effects (font (size 1.27 1.27)) (justify left))
-    )
-    (property "Footprint" "" (id 2) (at 205.74 80.01 0)
+    (property "Value" "HC-SR04" (id 1) (at 216.662 82.423 0)
+      (effects (font (size 1.27 1.27)) (justify left))
+    )
+    (property "Footprint" "XCVR_HC-SR04" (id 2) (at 205.74 80.01 0)
       (effects (font (size 1.27 1.27)) (justify left bottom) hide)
     )
@@
       (effects (font (size 1.27 1.27)) (justify left))
     )
-    (property "Value" "" (id 1) (at 216.662 98.933 0)
-      (effects (font (size 1.27 1.27)) (justify left))
-    )
-    (property "Footprint" "" (id 2) (at 205.74 96.52 0)
+    (property "Value" "HC-SR04" (id 1) (at 216.662 98.933 0)
+      (effects (font (size 1.27 1.27)) (justify left))
+    )
+    (property "Footprint" "XCVR_HC-SR04" (id 2) (at 205.74 96.52 0)
       (effects (font (size 1.27 1.27)) (justify left bottom) hide)
     )
@@
       (effects (font (size 1.27 1.27)) (justify left))
     )
-    (property "Value" "" (id 1) (at 216.662 115.443 0)
-      (effects (font (size 1.27 1.27)) (justify left))
-    )
-    (property "Footprint" "" (id 2) (at 205.74 113.03 0)
+    (property "Value" "HC-SR04" (id 1) (at 216.662 115.443 0)
+      (effects (font (size 1.27 1.27)) (justify left))
+    )
+    (property "Footprint" "XCVR_HC-SR04" (id 2) (at 205.74 113.03 0)
       (effects (font (size 1.27 1.27)) (justify left bottom) hide)
     )
@@
       (effects (font (size 1.27 1.27)) hide)
     )
-    (property "Value" "" (id 1) (at 200.787 122.5042 0))
+    (property "Value" "GNDREF" (id 1) (at 200.787 122.5042 0))
     (property "Footprint" "" (id 2) (at 200.66 118.11 0)
       (effects (font (size 1.27 1.27)) hide)
@@
       (effects (font (size 1.27 1.27)) hide)
     )
-    (property "Value" "" (id 1) (at 200.787 105.9942 0))
+    (property "Value" "GNDREF" (id 1) (at 200.787 105.9942 0))
     (property "Footprint" "" (id 2) (at 200.66 101.6 0)
       (effects (font (size 1.27 1.27)) hide)
@@
       (effects (font (size 1.27 1.27)) hide)
     )
-    (property "Value" "" (id 1) (at 200.787 89.4842 0))
+    (property "Value" "GNDREF" (id 1) (at 200.787 89.4842 0))
     (property "Footprint" "" (id 2) (at 200.66 85.09 0)
       (effects (font (size 1.27 1.27)) hide)
@@
       (effects (font (size 1.27 1.27)) hide)
     )
-    (property "Value" "" (id 1) (at 111.887 113.6142 0))
+    (property "Value" "GNDREF" (id 1) (at 111.887 113.6142 0))
     (property "Footprint" "" (id 2) (at 111.76 109.22 0)
       (effects (font (size 1.27 1.27)) hide)
@@
       (effects (font (size 1.27 1.27)) hide)
     )
-    (property "Value" "" (id 1) (at 163.1188 65.659 90)
+    (property "Value" "+5V" (id 1) (at 163.1188 65.659 90)
       (effects (font (size 1.27 1.27)) (justify left))
     )
@@
       (effects (font (size 1.27 1.27)) hide)
     )
-    (property "Value" "" (id 1) (at 197.4088 110.109 90)
+    (property "Value" "+5V" (id 1) (at 197.4088 110.109 90)
       (effects (font (size 1.27 1.27)) (justify left))
     )
@@
       (effects (font (size 1.27 1.27)) hide)
     )
-    (property "Value" "" (id 1) (at 197.4088 93.599 90)
+    (property "Value" "+5V" (id 1) (at 197.4088 93.599 90)
       (effects (font (size 1.27 1.27)) (justify left))
     )
@@
       (effects (font (size 1.27 1.27)) hide)
     )
-    (property "Value" "" (id 1) (at 197.4088 77.089 90)
+    (property "Value" "+5V" (id 1) (at 197.4088 77.089 90)
       (effects (font (size 1.27 1.27)) (justify left))
     )
@@
       (effects (font (size 1.27 1.27)) hide)
     )
-    (property "Value" "" (id 1) (at 92.71 82.55 90)
+    (property "Value" "GNDREF" (id 1) (at 92.71 82.55 90)
       (effects (font (size 1.27 1.27)) (justify right))
     )
@@
       (effects (font (size 1.27 1.27)) hide)
     )
-    (property "Value" "" (id 1) (at 169.037 123.7742 0))
+    (property "Value" "GNDREF" (id 1) (at 169.037 123.7742 0))
     (property "Footprint" "" (id 2) (at 168.91 119.38 0)
       (effects (font (size 1.27 1.27)) hide)
